Commit message: changed joint names in urdf A

File: bimanual_ws/src/Bimanual_Robot_Project_MuJoCo/allegro_hand_ros_v5/src/allegro_hand_description/allegro_hand_description_right_A.urdf (robot description, URDF)
Before this commit: robot allegro_hand_right, 22 links, 21 joints
Joints:
- removed joint joint_0_0
- removed joint joint_10_0
- removed joint joint_11_0
- removed joint joint_11_0_tip
- removed joint joint_12_0
- removed joint joint_14_0
- removed joint joint_15_0_tip
- removed joint joint_2_0
- removed joint joint_3_0
- removed joint joint_3_0_tip
- removed joint joint_5_0
- removed joint joint_7_0
- removed joint joint_8_0
- added joint right_joint_0_0: type revolute, parent palm_link, child link_0_0, origin xyz=0.00 0.0405 -0.00945 rpy=-0.08726646255 0 0, axis 0 0 1, limit lower=-0.47 upper=0.47 effort=15 velocity=7
- added joint right_joint_10_0: type revolute, parent link_9_0, child link_10_0, origin xyz=0 0 0.051, axis 0 1 0, limit lower=-0.174 upper=1.709 effort=15 velocity=7
- added joint right_joint_11_0: type revolute, parent link_10_0, child link_11_0, origin xyz=0 0 0.0384, axis 0 1 0, limit lower=-0.227 upper=1.618 effort=15 velocity=7
- added joint right_joint_11_0_tip: type fixed, parent link_11_0, child link_11_0_tip, origin xyz=0 0 0.0267 rpy=0 0 0
- added joint right_joint_12_0: type revolute, parent palm_link, child link_12_0, origin xyz=0.002 0.027 -0.06342 rpy=0 -1.65806278845 -1.5707963259, axis -1 0 0, limit lower=0.00 upper=1.78 effort=15 velocity=7
- added joint right_joint_14_0: type revolute, parent link_13_0, child link_14_0, origin xyz=0 0 0.00, axis 0 1 0, limit lower=-0.05 upper=1.85 effort=15 velocity=7
- added joint right_joint_15_0_tip: type fixed, parent link_15_0, child link_15_0_tip, origin xyz=0 0 0.05 rpy=0 0 0
- added joint right_joint_2_0: type revolute, parent link_1_0, child link_2_0, origin xyz=0 0 0.051, axis 0 1 0, limit lower=-0.174 upper=1.709 effort=15 velocity=7
- added joint right_joint_3_0: type revolute, parent link_2_0, child link_3_0, origin xyz=0 0 0.0384, axis 0 1 0, limit lower=-0.227 upper=1.618 effort=15 velocity=7
- added joint right_joint_3_0_tip: type fixed, parent link_3_0, child link_3_0_tip, origin xyz=0 0 0.0267 rpy=0 0 0
- added joint right_joint_5_0: type revolute, parent link_4_0, child link_5_0, origin xyz=0 0 0.021, axis 0 1 0, limit lower=-0.196 upper=1.8 effort=15 velocity=7
- added joint right_joint_7_0: type revolute, parent link_6_0, child link_7_0, origin xyz=0 0 0.0384, axis 0 1 0, limit lower=-0.227 upper=1.618 effort=15 velocity=7
- added joint right_joint_8_0: type revolute, parent palm_link, child link_8_0, origin xyz=0.0025 -0.0405 -0.00945 rpy=0.08726646255 0 0, axis 0 0 1, limit lower=-0.47 upper=0.47 effort=15 velocity=7

Commit message: updated all the values to move right arm and fingers

File: bimanual_ws/src/Bimanual_Robot_Project_MuJoCo/allegro_hand_ros_v5/src/allegro_hand_description/allegro_hand_description_right_A.urdf (robot description, URDF)
Before this commit: robot allegro_hand_right, 22 links, 21 joints
Links:
- removed link link_0_0
- removed link link_10_0
- removed link link_11_0
- removed link link_11_0_tip
- removed link link_12_0
- removed link link_13_0
- removed link link_14_0
- removed link link_15_0
- removed link link_15_0_tip
- removed link link_1_0
- removed link link_2_0
- removed link link_3_0
- removed link link_3_0_tip
- removed link link_4_0
- removed link link_5_0
- removed link link_6_0
- removed link link_7_0
- removed link link_7_0_tip
- removed link link_8_0
- removed link link_9_0
- removed link palm_link
- removed link world
- added link right_link_0_0, mass 0.0176; collision mesh filename=package://allegro_hand_description/meshes/l1.stl scale=0.001 0.001 0.001; visual mesh filename=package://allegro_hand_description/meshes/l1.stl scale=0.001 0.001 0.001
- added link right_link_10_0, mass 0.0366; collision mesh filename=package://allegro_hand_description/meshes/l3.stl scale=0.001 0.001 0.001; visual mesh filename=package://allegro_hand_description/meshes/l3.stl scale=0.001 0.001 0.001
- added link right_link_11_0, mass 0.00569; collision mesh filename=package://allegro_hand_description/meshes/l4.stl scale=0.001 0.001 0.001; visual mesh filename=package://allegro_hand_description/meshes/l4.stl scale=0.001 0.001 0.001
- added link right_link_11_0_tip, mass 0.00; collision mesh filename=package://allegro_hand_description/meshes/finger_tip.stl scale=0.001 0.001 0.001; visual mesh filename=package://allegro_hand_description/meshes/finger_tip.stl scale=0.001 0.001 0.001
- added link right_link_12_0, mass 0.0446; collision mesh filename=package://allegro_hand_description/meshes/t1_set.stl scale=0.001 0.001 0.001; visual mesh filename=package://allegro_hand_description/meshes/t1_set.stl scale=0.001 0.001 0.001
- added link right_link_13_0, mass 0.0173; collision mesh filename=package://allegro_hand_description/meshes/t2_set.stl scale=0.001 0.001 0.001; visual mesh filename=package://allegro_hand_description/meshes/t2_set.stl scale=0.001 0.001 0.001
- added link right_link_14_0, mass 0.03607; collision mesh filename=package://allegro_hand_description/meshes/t3_set.stl scale=0.001 0.001 0.001; visual mesh filename=package://allegro_hand_description/meshes/t3_set.stl scale=0.001 0.001 0.001
- added link right_link_15_0, mass 0.0338; collision mesh filename=package://allegro_hand_description/meshes/t4_set.stl scale=0.001 0.001 0.001; visual mesh filename=package://allegro_hand_description/meshes/t4_set.stl scale=0.001 0.001 0.001
- added link right_link_15_0_tip, mass 0.00; collision mesh filename=package://allegro_hand_description/meshes/finger_tip_silico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 scale=0.001 0.001 0.001; visual mesh filename=package://allegro_hand_description/meshes/finger_tip_silico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 scale=0.001 0.001 0.001
- added link right_link_1_0, mass 0.066; collision mesh filename=package://allegro_hand_description/meshes/l2.stl scale=0.001 0.001 0.001; visual mesh filename=package://allegro_hand_description/meshes/l2.stl scale=0.001 0.001 0.001
- added link right_link_2_0, mass 0.0366; collision mesh filename=package://allegro_hand_description/meshes/l3.stl scale=0.001 0.001 0.001; visual mesh filename=package://allegro_hand_description/meshes/l3.stl scale=0.001 0.001 0.001
- added link right_link_3_0, mass 0.00569; collision mesh filename=package://allegro_hand_description/meshes/l4.stl scale=0.001 0.001 0.001; visual mesh filename=package://allegro_hand_description/meshes/l4.stl scale=0.001 0.001 0.001
- added link right_link_3_0_tip, mass 0.00; collision mesh filename=package://allegro_hand_description/meshes/finger_tip.stl scale=0.001 0.001 0.001; visual mesh filename=package://allegro_hand_description/meshes/finger_tip.stl scale=0.001 0.001 0.001
- added link right_link_4_0, mass 0.0176; collision mesh filename=package://allegro_hand_description/meshes/l1.stl scale=0.001 0.001 0.001; visual mesh filename=package://allegro_hand_description/meshes/l1.stl scale=0.001 0.001 0.001
- added link right_link_5_0, mass 0.066; collision mesh filename=package://allegro_hand_description/meshes/l2.stl scale=0.001 0.001 0.001; visual mesh filename=package://allegro_hand_description/meshes/l2.stl scale=0.001 0.001 0.001
- added link right_link_6_0, mass 0.0366; collision mesh filename=package://allegro_hand_description/meshes/l3.stl scale=0.001 0.001 0.001; visual mesh filename=package://allegro_hand_description/meshes/l3.stl scale=0.001 0.001 0.001
- added link right_link_7_0, mass 0.00569; collision mesh filename=package://allegro_hand_description/meshes/l4.stl scale=0.001 0.001 0.001; visual mesh filename=package://allegro_hand_description/meshes/l4.stl scale=0.001 0.001 0.001
- added link right_link_7_0_tip, mass 0.00; collision mesh filename=package://allegro_hand_description/meshes/finger_tip.stl scale=0.001 0.001 0.001; visual mesh filename=package://allegro_hand_description/meshes/finger_tip.stl scale=0.001 0.001 0.001
- added link right_link_8_0, mass 0.0176; collision mesh filename=package://allegro_hand_description/meshes/l1.stl scale=0.001 0.001 0.001; visual mesh filename=package://allegro_hand_description/meshes/l1.stl scale=0.001 0.001 0.001
- added link right_link_9_0, mass 0.066; collision mesh filename=package://allegro_hand_description/meshes/l2.stl scale=0.001 0.001 0.001; visual mesh filename=package://allegro_hand_description/meshes/l2.stl scale=0.001 0.001 0.001
- added link right_palm_link, mass 0.4154; collision mesh filename=package://allegro_hand_description/meshes/palm.stl scale=0.001 0.001 0.001; visual mesh filename=package://allegro_hand_description/meshes/palm.stl scale=0.001 0.001 0.001
Joints:
- removed joint global
- removed joint joint_13_0
- removed joint joint_15_0
- removed joint joint_1_0
- removed joint joint_4_0
- removed joint joint_6_0
- removed joint joint_7_0_tip
- removed joint joint_9_0
- added joint right_joint_13_0: type revolute, parent right_link_12_0, child right_link_13_0, origin xyz=-0.001 0.00 0.06874, axis 0 0 1, limit lower=-0.26 upper=1.78 effort=15 velocity=7
- added joint right_joint_15_0: type revolute, parent right_link_14_0, child right_link_15_0, origin xyz=0 0 0.038, axis 0 1 0, limit lower=-0.09 upper=1.80 effort=15 velocity=7
- added joint right_joint_1_0: type revolute, parent right_link_0_0, child right_link_1_0, origin xyz=0.00 0 0.021, axis 0 1 0, limit lower=-0.196 upper=1.8 effort=15 velocity=7
- added joint right_joint_4_0: type revolute, parent right_palm_link, child right_link_4_0, origin xyz=0 0.00 -0.0079 rpy=0.0 0 0, axis 0 0 1, limit lower=-0.47 upper=0.47 effort=15 velocity=7
- added joint right_joint_6_0: type revolute, parent right_link_5_0, child right_link_6_0, origin xyz=0 0 0.051, axis 0 1 0, limit lower=-0.174 upper=1.709 effort=15 velocity=7
- added joint right_joint_7_0_tip: type fixed, parent right_link_7_0, child right_link_7_0_tip, origin xyz=0 0 0.0267 rpy=0 0 0
- added joint right_joint_9_0: type revolute, parent right_link_8_0, child right_link_9_0, origin xyz=0 0 0.021, axis 0 1 0, limit lower=-0.196 upper=1.8 effort=15 velocity=7
- added joint right_palm_joint: type fixed, parent right_link8, child right_palm_link, origin xyz=0 0 0 rpy=0 0 0
- joint right_joint_0_0: child link_0_0 -> right_link_0_0; parent palm_link -> right_palm_link
- joint right_joint_10_0: child link_10_0 -> right_link_10_0; parent link_9_0 -> right_link_9_0
- joint right_joint_11_0: child link_11_0 -> right_link_11_0; parent link_10_0 -> right_link_10_0
- joint right_joint_11_0_tip: child link_11_0_tip -> right_link_11_0_tip; parent link_11_0 -> right_link_11_0
- joint right_joint_12_0: child link_12_0 -> right_link_12_0; parent palm_link -> right_palm_link
- joint right_joint_14_0: child link_14_0 -> right_link_14_0; parent link_13_0 -> right_link_13_0
- joint right_joint_15_0_tip: child link_15_0_tip -> right_link_15_0_tip; parent link_15_0 -> right_link_15_0
- joint right_joint_2_0: child link_2_0 -> right_link_2_0; parent link_1_0 -> right_link_1_0
- joint right_joint_3_0: child link_3_0 -> right_link_3_0; parent link_2_0 -> right_link_2_0
- joint right_joint_3_0_tip: child link_3_0_tip -> right_link_3_0_tip; parent link_3_0 -> right_link_3_0
- joint right_joint_5_0: child link_5_0 -> right_link_5_0; parent link_4_0 -> right_link_4_0
- joint right_joint_7_0: child link_7_0 -> right_link_7_0; parent link_6_0 -> right_link_6_0
- joint right_joint_8_0: child link_8_0 -> right_link_8_0; parent palm_link -> right_palm_link

File: bimanual_ws/src/Bimanual_Robot_Project_MuJoCo/urdf/bimanual_panda.urdf.xacro (robot description, xacro)
@@ -3,6 +3,6 @@
 <xacro:include filename="$(find franka_description)/robots/panda_arm.xacro"/>
 <xacro:include filename="$(find franka_description)/robots/utils.xacro"/>
-<xacro:include filename="$(find allegro_hand_ros_v5-3Finger)/src/allegro_hand_description_3F.urdf"/>
-<xacro:include filename="$(find allegro_hand_rosv5)/src/allegro_hand_description/allegro_hand_description_right_A.urdf"/>
+<xacro:include filename="$(find bimanual_robot_project_mujoco)/allegro_hand_ros_v5-3Finger/src/allegro_hand_description/allegro_hand_description_3F.urdf"/>
+<xacro:include filename="$(find bimanual_robot_project_mujoco)/allegro_hand_ros_v5/src/allegro_hand_description/allegro_hand_description_right_A.urdf"/>
 <link name="base">
 <visual>
@@ -45,13 +45,13 @@
 <xacro:transmission-franka-model arm_id="left" root="left_joint1" tip="left_joint8" />
 <!--Left Hand-->
-<xacro:gazebo-joint joint="left_joint_0_0" transmission="hardware_interface/PositionJointInterface"/>
-<xacro:gazebo-joint joint="left_joint_1_0" transmission="hardware_interface/PositionJointInterface"/>
-<xacro:gazebo-joint joint="left_joint_2_0" transmission="hardware_interface/PositionJointInterface"/>
-<xacro:gazebo-joint joint="left_joint_3_0" transmission="hardware_interface/PositionJointInterface"/>
-<xacro:gazebo-joint joint="left_joint_4_0" transmission="hardware_interface/PositionJointInterface"/>
-<xacro:gazebo-joint joint="left_joint_5_0" transmission="hardware_interface/PositionJointInterface"/>
-<xacro:gazebo-joint joint="left_joint_6_0" transmission="hardware_interface/PositionJointInterface"/>
-<xacro:gazebo-joint joint="left_joint_7_0" transmission="hardware_interface/PositionJointInterface"/>
-<xacro:gazebo-joint joint="left_joint_8_0" transmission="hardware_interface/PositionJointInterface"/>
+<xacro:gazebo-joint joint="joint_0_0" transmission="hardware_interface/PositionJointInterface"/>
+<xacro:gazebo-joint joint="joint_1_0" transmission="hardware_interface/PositionJointInterface"/>
+<xacro:gazebo-joint joint="joint_2_0" transmission="hardware_interface/PositionJointInterface"/>
+<xacro:gazebo-joint joint="joint_3_0" transmission="hardware_interface/PositionJointInterface"/>
+<xacro:gazebo-joint joint="joint_4_0" transmission="hardware_interface/PositionJointInterface"/>
+<xacro:gazebo-joint joint="joint_5_0" transmission="hardware_interface/PositionJointInterface"/>
+<xacro:gazebo-joint joint="joint_6_0" transmission="hardware_interface/PositionJointInterface"/>
+<xacro:gazebo-joint joint="joint_7_0" transmission="hardware_interface/PositionJointInterface"/>
+<xacro:gazebo-joint joint="joint_8_0" transmission="hardware_interface/PositionJointInterface"/>
 <!--Right Arm-->
 <xacro:panda_arm arm_id="right" connected_to="base" xyz="0 -0.5 1" safety_distance="0.03" gazebo="true"/>
